Commit message: Created nail_test.py and successfully got the nailgun working

File: tests/nailgun.urdf (robot description, URDF)
Before this commit: robot nailgun.urdf, 1 links, 0 joints
Links:
- link baseLink: geometry collision box size=.025 .025 .2; visual mesh filename=cube.obj scale=.025 .025 .2
