Commit message: Worked out angle interpolation and how to get smoother motions on the kuka arms

File: urdfs/nailgun.urdf (robot description, URDF)
Before this commit: robot nailgun.urdf, 1 links, 0 joints
Links:
- link baseLink: geometry collision box size=.025 .025 .3; visual mesh filename=cube.obj scale=.025 .025 .3
