Commit message: Got all the back/side panels working, but gripper clips through when trying to rotate, next Ill try to reduce the mass of the panels

File: urdfs/handle.urdf (robot description, URDF)
Before this commit: robot front.urdf, 1 links, 0 joints
Links:
- link baseLink: mass 0.001 -> 0.05; geometry collision box size=.025 .0914 .1; visual mesh filename=cube.obj scale=.025 .0914 .1
